Commit message: Setup IMU and LIDAR in env vars as specified in Husky docs

File: urdf/husky_extras.urdf.xacro (robot description, xacro)
@@ -1,20 +1,7 @@
-<robot>
-  <!-- IMU Properties -->
-  <xacro:property name="imu_enclosure_x_size" value="0.028" />
-  <xacro:property name="imu_enclosure_y_size" value="0.028" />
-  <xacro:property name="imu_enclosure_z_size" value="0.009" />
-  <!-- IMU Link is the standard mounting position for the UM7 IMU.-->
-  <!-- Can be modified with environment variables in /etc/ros/setup.bash NOT ANYMORE -->
-  <link name="imu_link"/>
-  <joint name="imu_joint" type="fixed">
-    <origin xyz="${0.291+imu_enclosure_x_size/2} 0 ${0.284-imu_enclosure_z_size/2}" rpy="$(optenv HUSKY_IMU_RPY 0 0 0)" />
-    <parent link="top_plate_rear_link" />
-    <child link="imu_link" />
-  </joint>
-  <gazebo reference="imu_link">
-  </gazebo>
+<?xml version="1.0"?>
+<robot name="husky" xmlns:xacro="http://ros.org/wiki/xacro">
   <link name="os_sensor"/>
   <joint name="os_sensor_joint" type="fixed">
-    <origin xyz="${0.291+imu_enclosure_x_size/2} 0 0.361925" rpy="$(optenv HUSKY_LIDAR_RPY 0 0 0)" />
+    <origin xyz="$(optenv HUSKY_LIDAR_XYZ 0 0 0)" rpy="$(optenv HUSKY_LIDAR_RPY 0 0 0)" />
     <parent link="top_plate_rear_link" />
     <child link="os_sensor" />

Commit message: Update with zero rate gyors command sent to IMU. Add coments to setup scripts and update urdf

File: urdf/husky_extras.urdf.xacro (robot description, xacro)
@@ -1,4 +1,8 @@
 <?xml version="1.0"?>
 <robot name="husky" xmlns:xacro="http://ros.org/wiki/xacro">
+  <!-- IMU Properties -->
+  <xacro:property name="imu_enclosure_x_size" value="0.028" />
+  <xacro:property name="imu_enclosure_y_size" value="0.028" />
+  <xacro:property name="imu_enclosure_z_size" value="0.009" />
   <link name="os_sensor"/>
   <joint name="os_sensor_joint" type="fixed">

Commit message: Update all functions. Add version of systemctl loading sensors and base (TBD)

File: urdf/husky_extras.urdf.xacro (robot description, xacro)
@@ -8,5 +8,5 @@
   <joint name="os_sensor_joint" type="fixed">
     <origin xyz="$(optenv HUSKY_LIDAR_XYZ 0 0 0)" rpy="$(optenv HUSKY_LIDAR_RPY 0 0 0)" />
-    <parent link="top_plate_rear_link" />
+    <parent link="top_plate_link" />
     <child link="os_sensor" />
   </joint>

Commit message: Update conky monitor. Add all systemctl for individual packages and update URDF and setup stuff

File: urdf/husky_extras.urdf.xacro (robot description, xacro)
@@ -15,6 +15,6 @@
   <link name="gps_link"/>
   <joint name="gps_joint" type="fixed">
-    <origin xyz="$(optenv HUSKY_GPS_XYZ 0.35 0 0.245)" rpy="$(optenv HUSKY_GPS_RPY 0 0 0)" />
-    <parent link="base_link" />
+    <origin xyz="$(optenv HUSKY_GPS_XYZ 0.08 0 0.245)" rpy="$(optenv HUSKY_GPS_RPY 0 0 0)" />
+    <parent link="top_plate_front_link" />
     <child link="gps_link" />
   </joint>
